File: microsensor.kicad_sch (KiCad schematic)
At the start: 22 parts, among them J1 ARM SWD, Q1 IRLML2244TRPBF, SW1 Control, U1 HDC2080, U2 RV-3028-C7, U3 NORA B206, Y1 32768

Commit message: Remove RV3028 (firmware will use GRTC)
Parts:
- removed U2: RV-3028-C7, Package_SON:MicroCrystal_C7_SON-8_1.5x3.2mm_P0.9mm, symbol Timer_RTC:RV-3028-C7
- added TP2, TP3: P1.13, TestPoint:TestPoint_Pad_1.5x1.5mm, symbol Connector:TestPoint
- BT0: value CR1225 -> CR2032
Connections:
- net +BATT: now also TP2.1
- net GND: now also TP3.1
- net ~{RTCINT}: no longer names the net of U3.G9 (P1.05)
- no-connect marks 23 -> 22

Commit message: Put TP together, minor refactors, added more dimensions
Parts:
- TP1: renamed from TP3; value P1.13 -> GND
- TP2: value P1.13 -> BAT
- TP3: renamed from TP1; value P1.13 -> TX
Connections:
- net TX: now reaches TP3.1, U3.J8 (P1.13)
Other:
- moved on the sheet: TP1, TP2, TP3
